File: board/uv_led_lamp/uv_led_lamp.kicad_pcb (KiCad board)
At the start: 2 copper layers, 100 x 100 mm, 120 parts

Commit message: 1
Parts:
- R1, R10, R15, R16, R2, R23, R3, R30, R4, R5, R6, R7, R8, R9: footprint Resistor_THT:R_Axial_DIN0309_L9.0mm_D3.2mm_P12.70mm_Horizontal -> Resistor_THT:R_Axial_DIN0207_L6.3mm_D2.5mm_P10.16mm_Horizontal; moved to B.Cu
- R11: renamed from R12; footprint Resistor_THT:R_Axial_DIN0309_L9.0mm_D3.2mm_P12.70mm_Horizontal -> Resistor_THT:R_Axial_DIN0207_L6.3mm_D2.5mm_P10.16mm_Horizontal; moved to B.Cu
- R12: renamed from R14; footprint Resistor_THT:R_Axial_DIN0309_L9.0mm_D3.2mm_P12.70mm_Horizontal -> Resistor_THT:R_Axial_DIN0207_L6.3mm_D2.5mm_P10.16mm_Horizontal; moved to B.Cu
- R13: renamed from R11; footprint Resistor_THT:R_Axial_DIN0309_L9.0mm_D3.2mm_P12.70mm_Horizontal -> Resistor_THT:R_Axial_DIN0207_L6.3mm_D2.5mm_P10.16mm_Horizontal; moved to B.Cu
- R14: renamed from R13; footprint Resistor_THT:R_Axial_DIN0309_L9.0mm_D3.2mm_P12.70mm_Horizontal -> Resistor_THT:R_Axial_DIN0207_L6.3mm_D2.5mm_P10.16mm_Horizontal; moved to B.Cu
- R17: renamed from R21; footprint Resistor_THT:R_Axial_DIN0309_L9.0mm_D3.2mm_P12.70mm_Horizontal -> Resistor_THT:R_Axial_DIN0207_L6.3mm_D2.5mm_P10.16mm_Horizontal; moved to B.Cu
- R18: renamed from R26; footprint Resistor_THT:R_Axial_DIN0309_L9.0mm_D3.2mm_P12.70mm_Horizontal -> Resistor_THT:R_Axial_DIN0207_L6.3mm_D2.5mm_P10.16mm_Horizontal; moved to B.Cu
- R19: renamed from R17; footprint Resistor_THT:R_Axial_DIN0309_L9.0mm_D3.2mm_P12.70mm_Horizontal -> Resistor_THT:R_Axial_DIN0207_L6.3mm_D2.5mm_P10.16mm_Horizontal; moved to B.Cu
- R20: renamed from R22; footprint Resistor_THT:R_Axial_DIN0309_L9.0mm_D3.2mm_P12.70mm_Horizontal -> Resistor_THT:R_Axial_DIN0207_L6.3mm_D2.5mm_P10.16mm_Horizontal; moved to B.Cu
- R21: renamed from R27; footprint Resistor_THT:R_Axial_DIN0309_L9.0mm_D3.2mm_P12.70mm_Horizontal -> Resistor_THT:R_Axial_DIN0207_L6.3mm_D2.5mm_P10.16mm_Horizontal; moved to B.Cu
- R22: renamed from R18; footprint Resistor_THT:R_Axial_DIN0309_L9.0mm_D3.2mm_P12.70mm_Horizontal -> Resistor_THT:R_Axial_DIN0207_L6.3mm_D2.5mm_P10.16mm_Horizontal; moved to B.Cu
- R24: renamed from R28; footprint Resistor_THT:R_Axial_DIN0309_L9.0mm_D3.2mm_P12.70mm_Horizontal -> Resistor_THT:R_Axial_DIN0207_L6.3mm_D2.5mm_P10.16mm_Horizontal; moved to B.Cu
- R25: renamed from R19; footprint Resistor_THT:R_Axial_DIN0309_L9.0mm_D3.2mm_P12.70mm_Horizontal -> Resistor_THT:R_Axial_DIN0207_L6.3mm_D2.5mm_P10.16mm_Horizontal; moved to B.Cu
- R26: renamed from R24; footprint Resistor_THT:R_Axial_DIN0309_L9.0mm_D3.2mm_P12.70mm_Horizontal -> Resistor_THT:R_Axial_DIN0207_L6.3mm_D2.5mm_P10.16mm_Horizontal; moved to B.Cu
- R27: renamed from R29; footprint Resistor_THT:R_Axial_DIN0309_L9.0mm_D3.2mm_P12.70mm_Horizontal -> Resistor_THT:R_Axial_DIN0207_L6.3mm_D2.5mm_P10.16mm_Horizontal; moved to B.Cu
- R28: renamed from R20; footprint Resistor_THT:R_Axial_DIN0309_L9.0mm_D3.2mm_P12.70mm_Horizontal -> Resistor_THT:R_Axial_DIN0207_L6.3mm_D2.5mm_P10.16mm_Horizontal; moved to B.Cu
- R29: renamed from R25; footprint Resistor_THT:R_Axial_DIN0309_L9.0mm_D3.2mm_P12.70mm_Horizontal -> Resistor_THT:R_Axial_DIN0207_L6.3mm_D2.5mm_P10.16mm_Horizontal; moved to B.Cu
- moved R9 211.9 mm to (250.2, 47.2), turned to 180 degrees
- moved R6 209.7 mm to (250.2, 36.8), turned to 180 degrees
- moved D27 192.1 mm to (255.5, 44.0), turned to 0 degrees
- moved D45 191.5 mm to (255.5, 64.8), turned to 0 degrees
- moved D90 191.0 mm to (255.5, 116.8), turned to 0 degrees
- moved D36 185.2 mm to (255.5, 54.4), turned to 0 degrees
- moved D81 183.8 mm to (255.5, 106.4), turned to 0 degrees
- moved D53 182.5 mm to (243.8, 75.2), turned to 0 degrees
- moved R12 179.7 mm to (250.2, 57.6), turned to 180 degrees
- moved D72 177.3 mm to (255.5, 96.0), turned to 0 degrees
- moved R15 176.8 mm to (250.2, 68.0), turned to 180 degrees
- moved R8 174.4 mm to (204.9, 47.2)
- moved D26 173.0 mm to (243.8, 44.0), turned to 0 degrees
- moved R5 171.7 mm to (204.9, 36.8)
- moved D63 171.4 mm to (255.5, 85.6), turned to 0 degrees
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- renumbered D30 to D29, D32 to D30, D34 to D31, D36 to D32, D38 to D33, D40 to D34, D42 to D35, D44 to D36, D29 to D37, D31 to D38, D33 to D39, D6 to D4, D35 to D40, D37 to D41, D39 to D42, D41 to D43, D43 to D44, D51 to D47, D56 to D48, D61 to D49, D66 to D50, D71 to D51, D76 to D52, D81 to D53, D86 to D54, D47 to D55, D52 to D56, D62 to D58, D67 to D59, D4 to D6, D72 to D60, D77 to D61, D82 to D62, D87 to D63, D48 to D64, D53 to D65, D58 to D66, D63 to D67, D73 to D69, D9 to D7, D78 to D70, D83 to D71, D88 to D72, D49 to D73, D54 to D74, D59 to D75, D64 to D76, D69 to D77, D74 to D78, D84 to D80, D89 to D81, D50 to D82, D55 to D83, D60 to D84, D65 to D85, D70 to D86, D75 to D87, D80 to D88, D85 to D89, D7 to D9
Routing:
- net +12V: track 0.00 -> 278.8 mm
- net Net-(D15-K): track 0.00 -> 10.2 mm
- net Net-(D7-K): track 0.00 -> 10.1 mm
- net Net-(D87-K): track 0.00 -> 10.1 mm
- net Net-(D10-K): track 0.00 -> 10.1 mm
- net Net-(D70-K): track 0.00 -> 10.1 mm
- net Net-(D61-K): track 0.00 -> 10.1 mm
- net Net-(D52-K): track 0.00 -> 10.1 mm
- net Net-(D43-K): track 0.00 -> 10.1 mm
- net Net-(D34-K): track 0.00 -> 10.1 mm
- net Net-(D25-K): track 0.00 -> 10.1 mm
- net Net-(D16-K): track 0.00 -> 10.1 mm
- net Net-(D1-K): track 0.00 -> 10.1 mm
- net Net-(D78-K): track 0.00 -> 10.0 mm
- net Net-(D42-K): track 0.00 -> 10.0 mm
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
Commit message: 1
Routing:
- added copper zone on B.Cu, net GND
